Commit message: error fix

File: python/social_bot/models/kuka_lwr_4plus_cam/model.urdf (robot description, URDF)
Before this commit: robot kuka_lwr_4plus, 10 links, 10 joints
Joints:
- removed joint left_wheel_hinge

Commit message: add camera

File: python/social_bot/models/kuka_lwr_4plus_cam/model.urdf (robot description, URDF)
Before this commit: robot kuka_lwr_4plus, 10 links, 9 joints
Joints:
- joint camera_joint: axis  -> (none); child  -> camera_link; origin (none) -> xyz=0 0 2 rpy=0 0 0; parent  -> world

Commit message: add cam link

File: python/social_bot/models/kuka_lwr_4plus_cam/model.urdf (robot description, URDF)
Before this commit: robot kuka_lwr_4plus, 10 links, 9 joints
Joints:
- joint camera_joint: axis (none) -> ; child camera_link -> ; origin xyz=0 0 2 rpy=0 0 0 -> (none); parent world -> 

Commit message: succ in adding one more joint

File: python/social_bot/models/kuka_lwr_4plus_cam/model.urdf (robot description, URDF)
Before this commit: robot kuka_lwr_4plus_cam, 10 links, 9 joints
Links:
- removed link camera_link
- added link lwr_arm_8_link, mass 0.2; collision mesh filename=model://kuka_lwr_4plus/meshes/arm_flanche.dae scale=100 100 100; visual mesh filename=model://kuka_lwr_4plus/meshes/arm_flanche.dae scale=200 100 100
- link lwr_arm_7_link: geometry collision mesh filename=model://kuka_lwr_4plus/meshes/arm_flanche.dae scale=100 100 100; visual mesh filename=model://kuka_lwr_4plus/meshes/arm_flanche.dae scale=200 100 100
Joints:
- removed joint camera_joint
- added joint lwr_arm_7_joint: type revolute, parent lwr_arm_7_link, child lwr_arm_8_link, origin xyz=0 0 0.078 rpy=0 0 0, axis 0 0 1, limit lower=-2.96705972839 upper=2.96705972839 effort=204 velocity=3.14159265359

Commit message: add box link

File: python/social_bot/models/kuka_lwr_4plus_cam/model.urdf (robot description, URDF)
Before this commit: robot kuka_lwr_4plus_cam, 10 links, 9 joints
Links:
- link lwr_arm_8_link: geometry visual box 

Commit message: camera link

File: python/social_bot/models/kuka_lwr_4plus_cam/model.urdf (robot description, URDF)
Before this commit: robot kuka_lwr_4plus_cam, 10 links, 9 joints
Links:
- removed link lwr_arm_8_link
- added link camera_link, mass 0.2; visual box 
Joints:
- joint lwr_arm_7_joint: child lwr_arm_8_link -> camera_link

Commit message: no sensor

File: python/social_bot/models/kuka_lwr_4plus_cam/model.urdf (robot description, URDF)
Before this commit: robot kuka_lwr_4plus_cam, 10 links, 9 joints
Joints:
- removed joint lwr_arm_7_joint
- added joint camera_joint: type fixed, parent world, child camera_link, origin xyz=0 0 0.078 rpy=0 0 0, axis 0 0 1
